File: electrical/PIE_Final_Project_Schematic.kicad_sch (KiCad schematic)
At the start: 10 parts, among them U2 MPU-9250

Commit message: Final electrical schematic
Parts:
- removed U1: ~, symbol pie:Battery_Connector_Cable
- removed U3, U7, U8: ~, symbol pie:ESC_Speed_Controller
- removed U4, U5, U6: ~, symbol pie:Motor
- added U1, U3, U4: ~, symbol PIE_Symbol_Libary:Nidec_Motors
Connections:
- net at U2.13 (VDD): now also A2.17 (3V3); no longer A2.27 (+5V)
- net GND: now reaches U9. (GND)
- net GND: now also U1. (PWM), U3. (PWM), U4. (PWM)
- net at A2.10 (D7): now also U1. (PWM)
- net at A2.12 (D9): now also U3. (PWM)
- net at A2.13 (D10): now also U3. (PWM)
- net at A2.14 (MOSI): now also U3. (PWM)
- net +5V: now reaches A2.30 (VIN)
- net at A2.5 (D2): now also U4. (PWM)
- net at A2.6 (D3): now also U4. (PWM)
- net at A2.7 (D4): now also U4. (PWM)
- net at A2.8 (D5): now also U1. (PWM)
- net at A2.9 (D6): now also U1. (PWM)
- new net +12V: U1. (PWM), U3. (PWM), U4. (PWM), U9. (GND)
- no-connect marks 24 -> 20
Other:
- note added: "Nidec Motor"
- note removed: "Battery Connector Cable"
- note removed: "Brushless Motor"
- note removed: "ESC Speed Controller"

Commit message: Final Electrical Schematic (Kicad file)
Parts:
- removed U3, U4: ~, symbol PIE_Symbol_Libary:Nidec_Motors
- added SW1: SW_Push, symbol Switch:SW_Push
- added U3: ~, symbol PIE_Symbol_Libary:xt-60
Connections:
- net +5V is gone; now on net +12V: A2.30 (VIN)
- net +12V: now also SW1.1; no longer U9. (GND)
- net GND: now also U3. (GND); no longer U9. (GND)
- net at A2.10 (D7): no longer U1. (PWM)
- net at A2.12 (D9): now also U1. (PWM)
- net at A2.6 (D3): now also U1. (PWM)
- net at A2.8 (D5): no longer U1. (PWM)
- new net: U3. (GND), U9. (GND) (x2)
- new net: SW1.2, U3. (GND)
- no-connect marks 20 -> 31
Other:
- note added: "xt-60"

Commit message: Add files via upload
Connections:
- new net: U3. (GND), U9. (GND)
Other:
- note added: "12V Lipo Battery 2200mAh"
- note removed: "3S Lipo Battery 5200mAh"
Changed lines of the file:
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@@
 		)
 	)
-	(text "3S Lipo Battery \n5200mAh"
+	(text "12V Lipo Battery \n2200mAh"
 		(exclude_from_sim no)
 		(at 133.35 137.16 90)
@@
 	)
 	(symbol
-		(lib_name "pie:3S_Lipo_Battery_5200mAh")
 		(lib_id "pie:3S_Lipo_Battery_5200mAh")
 		(at 137.16 129.54 90)
